Commit message: add ORBSLAM2 & cartographer

File: paintingrobot/paintingrobot_description/urdf/base/paintingrobot_description_witharm.urdf.xacro (robot description, xacro)
@@ -646,5 +646,5 @@
         </plugin>
     </gazebo>
-    <!-- position controller -->
+<!-- position controller -->
     <gazebo>
       <plugin name="base_controller" filename="libgazebo_ros_planar_move.so">
@@ -657,4 +657,17 @@
       </plugin>
     </gazebo>
+<!-- ground truth plugin-->
+    <gazebo>
+      <plugin name="p3d_base_controller" filename="libgazebo_ros_p3d.so">
+        <alwaysOn>true</alwaysOn>
+        <updateRate>50.0</updateRate>
+        <bodyName>base_link</bodyName>
+        <topicName>ground_truth/state</topicName>
+        <gaussianNoise>0.01</gaussianNoise>
+        <frameName>world</frameName>
+        <xyzOffsets>0 0 0</xyzOffsets>
+        <rpyOffsets>0 0 0</rpyOffsets>
+      </plugin>
+    </gazebo>
     <gazebo reference="base_footprint">
       <turnGravityOff>true</turnGravityOff>

File: paintingrobot/paintingrobot_description/urdf/paintingrobot_witharm.xacro (robot description, xacro)
@@ -8,5 +8,5 @@
     <xacro:include filename="$(find paintingrobot_description)/urdf/sensors/zed.xacro" />
 <!--load xianquzhe base-->
-    <xacro:paintingrobot/>
+<xacro:paintingrobot/>
   <link name="base_footprint"/>
     <joint name="planar_joint" type="fixed">
@@ -20,5 +20,5 @@
     <parent link= "rodclimbing_link2"/>
     <child link = "kinect_link" />
-    <origin xyz="0.1 0.0 0.5" rpy="0 0 0.0" />
+    <origin xyz="0.1 0.0 0.35" rpy="0 0 0.0" />
   </joint>
 <!--load lidar-->

File: paintingrobot/paintingrobot_description/urdf/sensors/kinect_gazebo.xacro (robot description, xacro)
@@ -37,5 +37,5 @@
                     <clip>
                         <near>0.05</near>
-                        <far>3.0</far>
+                        <far>20.0</far>
                     </clip>
                 </camera>

Commit message: 增加激光雷达插件

File: paintingrobot/paintingrobot_description/urdf/base/paintingrobot_description_witharm.urdf.xacro (robot description, xacro)
@@ -721,13 +721,4 @@
       <turnGravityOff>true</turnGravityOff>
     </gazebo>
-    <gazebo reference="kinect_link">
-      <turnGravityOff>true</turnGravityOff>
-    </gazebo>
-    <gazebo reference="kinect_frame_optical">
-      <turnGravityOff>true</turnGravityOff>
-    </gazebo>
-    <gazebo reference="laser_link">
-      <turnGravityOff>true</turnGravityOff>
-    </gazebo>
 </xacro:macro>
 </robot>

File: paintingrobot/paintingrobot_description/urdf/paintingrobot_witharm.xacro (robot description, xacro)
@@ -3,7 +3,7 @@
     <xacro:include filename="$(find paintingrobot_description)/urdf/base/paintingrobot_description_witharm.urdf.xacro" />
 <!--include sensors-->
-    <xacro:include filename="$(find paintingrobot_description)/urdf/sensors/kinect_gazebo.xacro" />
-    <xacro:include filename="$(find paintingrobot_description)/urdf/sensors/lidar_gazebo.xacro" />
-    <xacro:include filename="$(find paintingrobot_description)/urdf/sensors/camera_gazebo.xacro" />
+    <!-- <xacro:include filename="$(find paintingrobot_description)/urdf/sensors/kinect_gazebo.xacro" /> -->
+    <!-- <xacro:include filename="$(find paintingrobot_description)/urdf/sensors/lidar_gazebo.xacro" /> -->
+    <!-- <xacro:include filename="$(find paintingrobot_description)/urdf/sensors/camera_gazebo.xacro" /> -->
     <xacro:include filename="$(find paintingrobot_description)/urdf/sensors/zed.xacro" />
 <!--load xianquzhe base-->
@@ -16,17 +16,17 @@
     </joint>
 <!--load kinect-->
-<xacro:kinect_camera prefix="kinect"  />
+<!-- <xacro:kinect_camera prefix="kinect"  />
   <joint name="kinect_joint" type="fixed">
     <parent link= "rodclimbing_link2"/>
     <child link = "kinect_link" />
     <origin xyz="0.1 0.0 0.35" rpy="0 0 0.0" />
-  </joint>
+  </joint> -->
 <!--load lidar-->
-<xacro:rplidar prefix="laser"  />
+<!-- <xacro:rplidar prefix="laser"  />
   <joint name="laser_joint" type="fixed">
     <parent link= "mobilebase_link"/>
     <child link = "laser_link" />
     <origin xyz="0.055 0.0 0.95" rpy="0.0 0.0 0.0" />
-  </joint>
+  </joint> -->
 <!--load zed-->
 <xacro:zed prefix="zed"  />
@@ -36,3 +36,32 @@
     <origin xyz="0.0 0.0 0.0" rpy="0.0 ${-M_PI/2} ${-M_PI/2}" />
   </joint>
+<!--load vlp_16-->
+  <!-- Parameters
+  *origin   URDF transform from parent link.
+  parent  URDF parent link name. Default base_link
+  name  URDF model name. Also used as tf frame_id for PointCloud2 output. Default velodyne
+  topic   PointCloud2 output topic name. Default /velodyne_points
+  hz Update   rate in hz. Default 10
+  lasers  Number of vertical spinning lasers. Default VLP-16: 16, HDL-32E: 32
+  samples Nuber of horizontal rotating samples. Default VLP-16: 1875, HDL-32E: 2187
+  min_range Minimum range value in meters. Default 0.9
+  max_range Maximum range value in meters. Default 130.0
+  noise Gausian noise value in meters. Default 0.008
+  min_angle Minimum horizontal angle in radians. Default -3.14
+  max_angle Maximum horizontal angle in radians. Default 3.14
+  gpu Use gpu_ray sensor instead of the standard ray sensor. Default false
+  min_intensity The minimum intensity beneath which returns will be clipped. Can be used to remove low-intensity objects.
+  -->
+<xacro:include filename="$(find paintingrobot_description)/urdf/sensors/VLP-16.urdf.xacro"/>
+  <VLP-16
+    parent="rodclimbing_link2"
+    hz="1"
+    lasers="64"
+    samples="2000"
+    min_range="0.9"
+    max_range="130.0"
+    min_angle="-${M_PI}"
+    max_angle="${M_PI}" >
+    <origin xyz="0.2 0 0.3" rpy="0 0 ${M_PI/2}" />
+  </VLP-16>
 </robot>
