Commit message: 模拟全站仪,八叉树建图

File: paintingrobot/paintingrobot_description/urdf/paintingrobot_witharm.xacro (robot description, xacro)
@@ -1,67 +1,79 @@
 <?xml version="1.0"?>
-<robot name="paintingrobot_witharm" xmlns:xacro="http://www.ros.org/wiki/xacro">
-    <xacro:include filename="$(find paintingrobot_description)/urdf/base/paintingrobot_description_witharm.urdf.xacro" />
-<!--include sensors-->
-    <!-- <xacro:include filename="$(find paintingrobot_description)/urdf/sensors/kinect_gazebo.xacro" /> -->
-    <!-- <xacro:include filename="$(find paintingrobot_description)/urdf/sensors/lidar_gazebo.xacro" /> -->
-    <!-- <xacro:include filename="$(find paintingrobot_description)/urdf/sensors/camera_gazebo.xacro" /> -->
-    <xacro:include filename="$(find paintingrobot_description)/urdf/sensors/zed.xacro" />
-<!--load xianquzhe base-->
-<xacro:paintingrobot/>
+<robot name="paintingrobot_witharm"
+  xmlns:xacro="http://www.ros.org/wiki/xacro">
+  <xacro:property name="PI" value="3.1415926"/>
+  <!-- include arm -->
+  <xacro:include filename="$(find paintingrobot_description)/urdf/base/paintingrobot_description_witharm.urdf.xacro" />
+  <!--include sensors-->
+  <!-- <xacro:include filename="$(find paintingrobot_description)/urdf/sensors/kinect_gazebo.xacro" /> -->
+  <xacro:include filename="$(find paintingrobot_description)/urdf/sensors/lidar_gazebo.xacro" />
+  <!-- <xacro:include filename="$(find paintingrobot_description)/urdf/sensors/camera_gazebo.xacro" /> -->
+  <!-- <xacro:include filename="$(find paintingrobot_description)/urdf/sensors/zed.xacro" /> -->
+  <!-- 3个Kinect仿真全站仪 -->
+  <xacro:include filename="$(find paintingrobot_description)/urdf/sensors/kinect_1_gazebo.xacro" />
+  <xacro:include filename="$(find paintingrobot_description)/urdf/sensors/kinect_2_gazebo.xacro" />
+  <xacro:include filename="$(find paintingrobot_description)/urdf/sensors/kinect_3_gazebo.xacro" />
+  <!--load xianquzhe base-->
+  <xacro:paintingrobot/>
   <link name="base_footprint"/>
-    <joint name="planar_joint" type="fixed">
-      <origin xyz="0 0 0" rpy="0 0 0"/>
-      <parent link="base_footprint"/>
-      <child link="base_link"/>
-    </joint>
-<!--load kinect-->
-<!-- <xacro:kinect_camera prefix="kinect"  />
-  <joint name="kinect_joint" type="fixed">
-    <parent link= "rodclimbing_link2"/>
-    <child link = "kinect_link" />
-    <origin xyz="0.1 0.0 0.35" rpy="0 0 0.0" />
-  </joint> -->
-<!--load lidar-->
-<!-- <xacro:rplidar prefix="laser"  />
+  <joint name="planar_joint" type="fixed">
+    <origin xyz="0 0 0" rpy="0 0 0"/>
+    <parent link="base_footprint"/>
+    <child link="base_link"/>
+  </joint>
+  <!--load kinect_1-->
+  <xacro:kinect_camera_1 prefix="kinect_1"/>
+  <joint name="kinect_joint_1" type="fixed">
+    <parent link= "mobilebase_link"/>
+    <child link = "kinect_1_link" />
+    <origin xyz="0.5 0.0 1" rpy="0 0 0.0" />
+  </joint>
+  <!--load kinect_2-->
+  <xacro:kinect_camera_2 prefix="kinect_2"/>
+  <joint name="kinect_joint_2" type="fixed">
+    <parent link= "mobilebase_link"/>
+    <child link = "kinect_2_link" />
+    <origin xyz="0.5 0 1" rpy="0 0 ${PI*2/3}" />
+  </joint>
+  <!--load kinect_3-->
+  <xacro:kinect_camera_3 prefix="kinect_3"/>
+  <joint name="kinect_joint_3" type="fixed">
+    <parent link= "mobilebase_link"/>
+    <child link = "kinect_3_link" />
+    <origin xyz="0.5 0 1" rpy="0 0 ${PI*4/3}" />
+  </joint>
+  <!--load lidar-->
+  <xacro:rplidar prefix="laser" />
   <joint name="laser_joint" type="fixed">
     <parent link= "mobilebase_link"/>
     <child link = "laser_link" />
     <origin xyz="0.055 0.0 0.95" rpy="0.0 0.0 0.0" />
-  </joint> -->
-<!--load zed-->
-<xacro:zed prefix="zed"  />
+  </joint>
+  <!--load zed-->
+  <!-- <xacro:zed prefix="zed" />
   <joint name="zed_joint" type="fixed">
     <parent link= "wrist3_Link"/>
     <child link = "zed_camera_center" />
     <origin xyz="0.0 0.0 0.0" rpy="0.0 ${-M_PI/2} ${-M_PI/2}" />
-  </joint>
-<!--load vlp_16-->
+  </joint> -->
+  <!-- load VLP-16 -->
   <!-- Parameters
-  *origin   URDF transform from parent link.
-  parent  URDF parent link name. Default base_link
-  name  URDF model name. Also used as tf frame_id for PointCloud2 output. Default velodyne
-  topic   PointCloud2 output topic name. Default /velodyne_points
-  hz Update   rate in hz. Default 10
-  lasers  Number of vertical spinning lasers. Default VLP-16: 16, HDL-32E: 32
-  samples Nuber of horizontal rotating samples. Default VLP-16: 1875, HDL-32E: 2187
-  min_range Minimum range value in meters. Default 0.9
-  max_range Maximum range value in meters. Default 130.0
-  noise Gausian noise value in meters. Default 0.008
-  min_angle Minimum horizontal angle in radians. Default -3.14
-  max_angle Maximum horizontal angle in radians. Default 3.14
-  gpu Use gpu_ray sensor instead of the standard ray sensor. Default false
-  min_intensity The minimum intensity beneath which returns will be clipped. Can be used to remove low-intensity objects.
-  -->
-<xacro:include filename="$(find paintingrobot_description)/urdf/sensors/VLP-16.urdf.xacro"/>
-  <VLP-16
-    parent="rodclimbing_link2"
-    hz="1"
-    lasers="64"
-    samples="2000"
-    min_range="0.9"
-    max_range="130.0"
-    min_angle="-${M_PI}"
-    max_angle="${M_PI}" >
+    *origin   URDF transform from parent link.
+    parent  URDF parent link name. Default base_link
+    name  URDF model name. Also used as tf frame_id for PointCloud2 output. Default velodyne
+    topic   PointCloud2 output topic name. Default /velodyne_points
+    hz Update   rate in hz. Default 10
+    lasers  Number of vertical spinning lasers. Default VLP-16: 16, HDL-32E: 32
+    samples Nuber of horizontal rotating samples. Default VLP-16: 1875, HDL-32E: 2187
+    min_range Minimum range value in meters. Default 0.9
+    max_range Maximum range value in meters. Default 130.0
+    noise Gausian noise value in meters. Default 0.008
+    min_angle Minimum horizontal angle in radians. Default -3.14
+    max_angle Maximum horizontal angle in radians. Default 3.14
+    gpu Use gpu_ray sensor instead of the standard ray sensor. Default false
+    min_intensity The minimum intensity beneath which returns will be clipped. Can be used to remove low-intensity objects.-->
+  <!-- <xacro:include filename="$(find paintingrobot_description)/urdf/sensors/VLP-16.urdf.xacro"/>
+  <VLP-16 parent="rodclimbing_link2" hz="1" lasers="64" samples="2000" min_range="0.9" max_range="130.0" min_angle="-${M_PI}" max_angle="${M_PI}">
     <origin xyz="0.2 0 0.3" rpy="0 0 ${M_PI/2}" />
-  </VLP-16>
+  </VLP-16> -->
 </robot>

File: paintingrobot/paintingrobot_description/urdf/sensors/kinect_gazebo.xacro (robot description, xacro)
@@ -29,5 +29,5 @@
                 <update_rate>20.0</update_rate>
                 <camera>
-                    <horizontal_fov>${60.0*M_PI/180.0}</horizontal_fov>
+                    <horizontal_fov>${120.0*M_PI/180.0}</horizontal_fov>
                     <image>
                         <format>R8G8B8</format>
@@ -52,5 +52,5 @@
                     <frameName>${prefix}_frame_optical</frameName>
                     <pointCloudCutoff>0.5</pointCloudCutoff>
-                    <pointCloudCutoffMax>3.0</pointCloudCutoffMax>
+                    <pointCloudCutoffMax>10</pointCloudCutoffMax>
                     <distortionK1>0.00000001</distortionK1>
                     <distortionK2>0.00000001</distortionK2>
